Commit message: Add files via upload
Modified billi.xacro and corrected body.xacro

File: billi_sim/models/urdf/leg.xacro (robot description, xacro)
@@ -1,6 +1,7 @@
+<?xml version="1.0"?>
 <robot name="billi" xmlns:xacro="http://www.ros.org/wiki/xacro">
-  <link name="leg">
+<link name="leg1">
     <visual>
-	<origin rpy="0 0 0" xyz="0 0 0"/>
+    	<origin rpy="0 0 0" xyz="0 0 0"/>
       <geometry>
         <mesh filename="package://billi_sim/models/meshes/leg1.stl" scale ="1 1 1"/>
@@ -18,6 +19,32 @@
 		  <inertia ixx="0.0395416666667" ixy="0" ixz="0" iyy="0.106208333333" iyz="0" izz="0.106208333333"/>
 		</inertial>
-  </link>
-<gazebo reference="leg">
+</link>
+<gazebo reference="leg1">
+        <kp>1000.0</kp>
+        <kd>1000.0</kd>
+        <mu1>10.0</mu1>
+        <mu2>10.0</mu2>
+        <material>Gazebo/blue</material>
+    </gazebo>
+ <link name="leg2">
+    <visual>
+	<origin rpy="0 0 0" xyz="5 5 5"/>
+      <geometry>
+        <mesh filename="package://billi_sim/models/meshes/leg2.stl" scale ="1 1 1"/>
+      </geometry>
+      <material name="blue"/>
+    </visual>
+    <collision>
+      <geometry>
+        <mesh filename="package://billi_sim/models/meshes/leg2.stl" scale ="1 1 1"/>
+      </geometry>
+    </collision>
+	<inertial>
+		  <mass value="1.0"/>
+		  <origin rpy="0 0 0" xyz="0 0 0.1"/>
+		  <inertia ixx="0.0395416666667" ixy="0" ixz="0" iyy="0.106208333333" iyz="0" izz="0.106208333333"/>
+		</inertial>
+   </link>
+<gazebo reference="leg2">
         <kp>1000.0</kp>
         <kd>1000.0</kd>
