Commit message: Merge by temporarily fixing conflicts (#7)

File: billi_sim/models/urdf/head.xacro (robot description, xacro)
@@ -3,7 +3,7 @@
    <link name="head">
     <visual>
-	<origin rpy="0 0 0" xyz="0 0 0"/>
+	<origin rpy="3.14 0 1" xyz="0 0 0"/>
       <geometry>
-        <mesh filename="package://billi_sim/meshes/head.stl" scale ="1 1 1"/>
+        <mesh filename="package://billi_sim/models/meshes/head.stl" scale ="1 1 1"/>
       </geometry>
       <material name="blue"/>
@@ -11,5 +11,5 @@
     <collision>
       <geometry>
-        <mesh filename="package://billi_sim/meshes/head.stl" scale ="1 1 1"/>
+        <mesh filename="package://billi_sim/models/meshes/head.stl" scale ="1 1 1"/>
       </geometry>
     </collision>
