Commit message: Explanative commit message

File: billi_sim/models/urdf/billi.xacro (robot description, xacro)
@@ -6,8 +6,17 @@
   <xacro:property name="d_tbb" value="0.082"/>
   <xacro:property name="d_p1p2" value="0.35"/>
+    <xacro:macro name="hyq_leg" params="name parent *origin reflect_hip reflect_upper reflect_front">
 	<!-- billi shoulder -->
 	<xacro:include filename="$(find billi_sim)/models/urdf/shoulder.xacro"/>
+    <xacro:include filename="$(find towr_simulator)/models/urdf/shoulder.xacro"/>
 	<!-- billi body -->
 	<xacro:include filename="$(find billi_sim)/models/urdf/body.xacro"/>
+    <xacro:include filename="$(find towr_simulator)/models/urdf/body.xacro"/>
+    <!-- billi leg -->
+	<xacro:include filename="$(find billi_sim)/models/urdf/leg.xacro"/>
+    <xacro:include filename="$(find towr_simulator)/models/urdf/leg.xacro"/>
+    <!-- billi head -->
+	<xacro:include filename="$(find billi_sim)/models/urdf/head.xacro"/>
+    <xacro:include filename="$(find towr_simulator)/models/urdf/head.xacro"/>
 	<gazebo>
 		<plugin name="gazebo_ros_control" filename="libgazebo_ros_control.so"/>
@@ -16,4 +25,68 @@
 	<!-- body -->
 	<xacro:billi_body name="base"/>
+    <joint name="lf_haa_joint" type="revolute">
+			<xacro:insert_block name="origin"/>
+			<parent link="base"/>
+			<child  link="lf_hipassembly"/>
+			<axis xyz="0 0 1"/>
+			<limit effort="150.0" velocity="12.0" lower="${-7*PI/18}" upper="${PI/6}"/>
+	</joint>
+    <joint name="lh_haa_joint" type="revolute">
+			<xacro:insert_block name="origin"/>
+			<parent link="base"/>
+			<child  link="lh_hipassembly"/>
+			<axis xyz="0 0 1"/>
+			<limit effort="150.0" velocity="12.0" lower="${-7*PI/18}" upper="${PI/6}"/>
+	</joint>
+    <joint name="rf_haa_joint" type="revolute">
+			<xacro:insert_block name="origin"/>
+			<parent link="base"/>
+			<child  link="rf_hipassembly"/>
+			<axis xyz="0 0 1"/>
+			<limit effort="150.0" velocity="12.0" lower="${-7*PI/18}" upper="${PI/6}"/>
+	</joint>
+    <joint name="rh_haa_joint" type="revolute">
+			<xacro:insert_block name="origin"/>
+			<parent link="base"/>
+			<child  link="rh_hipassembly"/>
+			<axis xyz="0 0 1"/>
+			<limit effort="150.0" velocity="12.0" lower="${-7*PI/18}" upper="${PI/6}"/>
+	</joint>
+    <joint name="lf_hfe_joint" type="revolute">
+			<origin xyz="${d_tbb} 0 0" rpy="${reflect_upper*PI/2} 0 0"/>
+			<parent link="lf_hipassembly"/>
+			<child  link="lf_upperleg"/>
+			<axis xyz="0 0 1"/>
+			<limit effort="150.0" velocity="12.0"
+          lower="${-(1+reflect_front)*5*PI/36-(1-reflect_front)*7*PI/36}"
+		  upper="${(1-reflect_front)*5*PI/36+(1+reflect_front)*7*PI/36}"/>
+	</joint>
+    <joint name="lh_hfe_joint" type="revolute">
+			<origin xyz="${d_tbb} 0 0" rpy="${reflect_upper*PI/2} 0 0"/>
+			<parent link="lh_hipassembly"/>
+			<child  link="lh_upperleg"/>
+			<axis xyz="0 0 1"/>
+			<limit effort="150.0" velocity="12.0"
+          lower="${-(1+reflect_front)*5*PI/36-(1-reflect_front)*7*PI/36}"
+		  upper="${(1-reflect_front)*5*PI/36+(1+reflect_front)*7*PI/36}"/>
+	</joint>
+    <joint name="rh_hfe_joint" type="revolute">
+			<origin xyz="${d_tbb} 0 0" rpy="${reflect_upper*PI/2} 0 0"/>
+			<parent link="rh_hipassembly"/>
+			<child  link="rh_upperleg"/>
+			<axis xyz="0 0 1"/>
+			<limit effort="150.0" velocity="12.0"
+          lower="${-(1+reflect_front)*5*PI/36-(1-reflect_front)*7*PI/36}"
+		  upper="${(1-reflect_front)*5*PI/36+(1+reflect_front)*7*PI/36}"/>
+	</joint>
+    <joint name="rf_hfe_joint" type="revolute">
+			<origin xyz="${d_tbb} 0 0" rpy="${reflect_upper*PI/2} 0 0"/>
+			<parent link="rf}_hipassembly"/>
+			<child  link="rf_upperleg"/>
+			<axis xyz="0 0 1"/>
+			<limit effort="150.0" velocity="12.0"
+          lower="${-(1+reflect_front)*5*PI/36-(1-reflect_front)*7*PI/36}"
+		  upper="${(1-reflect_front)*5*PI/36+(1+reflect_front)*7*PI/36}"/>
+	</joint>
 	<!-- front shoulder -->
 	<!--xacro:billi_shoulder
@@ -56,3 +129,4 @@
 		<xacro:trans num="1" name="fs" part="haa"/>
 		<xacro:trans num="2" name="bs" part="haa"/-->
+    </xacro:macro>
 </robot>

Commit message: Add files via upload

File: billi_sim/models/urdf/billi.xacro (robot description, xacro)
@@ -2,18 +2,96 @@
 <robot name="billi" xmlns:xacro="http://www.ros.org/wiki/xacro">
   <!-- billi shoulder -->
+<<<<<<< HEAD
+	<!--xacro:include filename="$(find billi_sim)/models/urdf/shoulder.xacro"/-->
+=======
 	<xacro:include filename="$(find billi_sim)/models/urdf/shoulder.xacro"/>
+>>>>>>> a2351546f9e6cd629167bb84ce18117092a4d7df
 	<!-- billi body -->
 	<xacro:include filename="$(find billi_sim)/models/urdf/body.xacro"/>
     <!-- billi leg -->
+<<<<<<< HEAD
+	<xacro:include filename="$(find billi_sim)/models/urdf/leg1.xacro"/>
+	<xacro:include filename="$(find billi_sim)/models/urdf/leg2.xacro"/>
+	<xacro:include filename="$(find billi_sim)/models/urdf/leg3.xacro"/>
+	<xacro:include filename="$(find billi_sim)/models/urdf/leg4.xacro"/>
+	<xacro:include filename="$(find billi_sim)/models/urdf/leg-lower4.xacro"/>
+	<xacro:include filename="$(find billi_sim)/models/urdf/leg-lower2.xacro"/>
+	<xacro:include filename="$(find billi_sim)/models/urdf/leg-lower1.xacro"/>
+	<xacro:include filename="$(find billi_sim)/models/urdf/leg-lower3.xacro"/>
+=======
 	<xacro:include filename="$(find billi_sim)/models/urdf/leg.xacro"/>
+>>>>>>> a2351546f9e6cd629167bb84ce18117092a4d7df
     <!-- billi head -->
 	<xacro:include filename="$(find billi_sim)/models/urdf/head.xacro"/>
+<<<<<<< HEAD
+	<!--gazebo>
+		<plugin name="gazebo_ros_control" filename="libgazebo_ros_control.so"/>
+	</gazebo-->
+=======
 	<gazebo>
 		<plugin name="gazebo_ros_control" filename="libgazebo_ros_control.so"/>
 	</gazebo>
+>>>>>>> a2351546f9e6cd629167bb84ce18117092a4d7df
 	<!-- body -->
 	<!-- <xacro:billi_body name="base"/> -->
+<<<<<<< HEAD
+<joint name="lower_upper1" type="revolute">
+			<origin xyz="0.0 -0.039282 0.0" rpy="0 0 0"/>
+			<parent link="leg1"/>
+			<child  link="leg-lower1"/>
+			<axis xyz="0 0 1"/>
+			<limit effort="150.0" velocity="12.0"
+          lower="-1.57"
+		  upper="1.57"/>
+	</joint>
+<gazebo reference="lower_upper1">
+		<provideFeedback>true</provideFeedback>
+		<disableFixedJointLumping>true</disableFixedJointLumping>
+		</gazebo>
+<joint name="lower_upper2" type="revolute">
+			<origin xyz="0.0 -0.039282 0.0" rpy="0 0 0"/>
+			<parent link="leg2"/>
+			<child  link="leg-lower2"/>
+			<axis xyz="0 0 1"/>
+			<limit effort="150.0" velocity="12.0"
+          lower="-1.57"
+		  upper="1.57"/>
+	</joint>
+<gazebo reference="lower_upper2">
+		<provideFeedback>true</provideFeedback>
+		<disableFixedJointLumping>true</disableFixedJointLumping>
+		</gazebo>
+<joint name="lower_upper4" type="revolute">
+			<origin xyz="0.0 -0.039282 0.0" rpy="0 0 0"/>
+			<parent link="leg4"/>
+			<child  link="leg-lower4"/>
+			<axis xyz="0 0 1"/>
+			<limit effort="150.0" velocity="12.0"
+          lower="-1.57"
+		  upper="1.57"/>
+	</joint>
+<gazebo reference="lower_upper4">
+		<provideFeedback>true</provideFeedback>
+		<disableFixedJointLumping>true</disableFixedJointLumping>
+		</gazebo>
+<joint name="lower_upper3" type="revolute">
+			<origin xyz="0.0 -0.039282 0.0" rpy="0 0 0"/>
+			<parent link="leg3"/>
+			<child  link="leg-lower3"/>
+			<axis xyz="0 0 1"/>
+			<limit effort="150.0" velocity="12.0"
+          lower="-1.57"
+		  upper="1.57"/>
+	</joint>
+<gazebo reference="lower_upper3">
+		<provideFeedback>true</provideFeedback>
+		<disableFixedJointLumping>true</disableFixedJointLumping>
+		</gazebo>
     <joint name="head_body" type="revolute">
-			<origin xyz="0 0 0" rpy="0 0 0"/>
+			<origin xyz="0.098 0.035 -0.048" rpy="0 0 0"/>
+=======
+    <joint name="head_body" type="revolute">
+			<origin xyz="0 0 0" rpy="0 0 0"/>
+>>>>>>> a2351546f9e6cd629167bb84ce18117092a4d7df
 			<parent link="body"/>
 			<child  link="head"/>
@@ -31,5 +109,9 @@
 			<parent link="body"/>
 			<child  link="leg1"/>
-			<axis xyz="1 0 0"/>
+<<<<<<< HEAD
+			<axis xyz="0 0 1"/>
+=======
+			<axis xyz="1 0 0"/>
+>>>>>>> a2351546f9e6cd629167bb84ce18117092a4d7df
 			<limit effort="150.0" velocity="12.0"
           lower="-1.57"
@@ -41,8 +123,15 @@
 		</gazebo>
    <joint name="left_hand" type="revolute">
+<<<<<<< HEAD
+			<origin xyz="0 0 -0.092" rpy="0 0 0"/>
+			<parent link="body"/>
+			<child  link="leg4"/>
+			<axis xyz="0 0 1"/>
+=======
 			<origin xyz="0 0 0" rpy="0 0 0"/>
 			<parent link="body"/>
 			<child  link="leg2"/>
 			<axis xyz="1 0 0"/>
+>>>>>>> a2351546f9e6cd629167bb84ce18117092a4d7df
 			<limit effort="150.0" velocity="12.0"
           lower="-1.57"
@@ -54,8 +143,15 @@
 		</gazebo>
  <joint name="right_leg" type="revolute">
+<<<<<<< HEAD
+			<origin xyz=".083 .017 0" rpy="0 0 0"/>
+			<parent link="body"/>
+			<child  link="leg2"/>
+			<axis xyz="0 0 1"/>
+=======
 			<origin xyz="0 0 0" rpy="0 0 0"/>
 			<parent link="body"/>
 			<child  link="leg1"/>
 			<axis xyz="1 0 0"/>
+>>>>>>> a2351546f9e6cd629167bb84ce18117092a4d7df
 			<limit effort="150.0" velocity="12.0"
           lower="-1.57"
@@ -67,8 +163,15 @@
 			</gazebo>
     <joint name="left_leg" type="revolute">
+<<<<<<< HEAD
+			<origin xyz="0.083 0.017 -0.092" rpy="0 0 0"/>
+			<parent link="body"/>
+			<child  link="leg3"/>
+			<axis xyz="0 0 1"/>
+=======
 			<origin xyz="0 0 0" rpy="0 0 0"/>
 			<parent link="body"/>
 			<child  link="leg2"/>
 			<axis xyz="1 0 0"/>
+>>>>>>> a2351546f9e6cd629167bb84ce18117092a4d7df
 			<limit effort="150.0" velocity="12.0"
           lower="-1.57"
@@ -79,3 +182,104 @@
 		<disableFixedJointLumping>true</disableFixedJointLumping>
 		</gazebo>
+<<<<<<< HEAD
+<!-- Adding transmissions-->
+<transmission name="head">
+    <type>transmission_interface/SimpleTransmission</type>
+    <joint name="head_body">
+      <hardwareInterface>hardware_interface/EffortJointInterface</hardwareInterface>
+    </joint>
+    <actuator name="motor_head">
+      <hardwareInterface>EffortJointInterface</hardwareInterface>
+      <mechanicalReduction>1</mechanicalReduction>
+    </actuator>
+  </transmission>
+<transmission name="lu1">
+    <type>transmission_interface/SimpleTransmission</type>
+    <joint name="right_hand">
+      <hardwareInterface>hardware_interface/EffortJointInterface</hardwareInterface>
+    </joint>
+    <actuator name="motor1">
+      <hardwareInterface>EffortJointInterface</hardwareInterface>
+      <mechanicalReduction>1</mechanicalReduction>
+    </actuator>
+  </transmission>
+<transmission name="lb1">
+    <type>transmission_interface/SimpleTransmission</type>
+    <joint name="lower_upper1">
+      <hardwareInterface>hardware_interface/EffortJointInterface</hardwareInterface>
+    </joint>
+    <actuator name="motor2">
+      <hardwareInterface>EffortJointInterface</hardwareInterface>
+      <mechanicalReduction>1</mechanicalReduction>
+    </actuator>
+  </transmission>
+<transmission name="lu2">
+    <type>transmission_interface/SimpleTransmission</type>
+    <joint name="right_leg">
+      <hardwareInterface>hardware_interface/EffortJointInterface</hardwareInterface>
+    </joint>
+    <actuator name="motor3">
+      <hardwareInterface>EffortJointInterface</hardwareInterface>
+      <mechanicalReduction>1</mechanicalReduction>
+    </actuator>
+  </transmission>
+<transmission name="lb2">
+    <type>transmission_interface/SimpleTransmission</type>
+    <joint name="lower_upper2">
+      <hardwareInterface>hardware_interface/EffortJointInterface</hardwareInterface>
+    </joint>
+    <actuator name="motor4">
+      <hardwareInterface>EffortJointInterface</hardwareInterface>
+      <mechanicalReduction>1</mechanicalReduction>
+    </actuator>
+  </transmission>
+<transmission name="lu3">
+    <type>transmission_interface/SimpleTransmission</type>
+    <joint name="left_leg">
+      <hardwareInterface>hardware_interface/EffortJointInterface</hardwareInterface>
+    </joint>
+    <actuator name="motor5">
+      <hardwareInterface>EffortJointInterface</hardwareInterface>
+      <mechanicalReduction>1</mechanicalReduction>
+    </actuator>
+  </transmission>
+<transmission name="lb3">
+    <type>transmission_interface/SimpleTransmission</type>
+    <joint name="lower_upper3">
+      <hardwareInterface>hardware_interface/EffortJointInterface</hardwareInterface>
+    </joint>
+    <actuator name="motor6">
+      <hardwareInterface>EffortJointInterface</hardwareInterface>
+      <mechanicalReduction>1</mechanicalReduction>
+    </actuator>
+  </transmission>
+<transmission name="lu4">
+    <type>transmission_interface/SimpleTransmission</type>
+    <joint name="left_hand">
+      <hardwareInterface>hardware_interface/EffortJointInterface</hardwareInterface>
+    </joint>
+    <actuator name="motor7">
+      <hardwareInterface>EffortJointInterface</hardwareInterface>
+      <mechanicalReduction>1</mechanicalReduction>
+    </actuator>
+  </transmission>
+<transmission name="lb4">
+    <type>transmission_interface/SimpleTransmission</type>
+    <joint name="lower_upper4">
+      <hardwareInterface>hardware_interface/EffortJointInterface</hardwareInterface>
+    </joint>
+    <actuator name="motor8">
+      <hardwareInterface>EffortJointInterface</hardwareInterface>
+      <mechanicalReduction>1</mechanicalReduction>
+    </actuator>
+  </transmission>
+<gazebo>
+  <plugin name="gazebo_ros_control" filename="libgazebo_ros_control.so">
+    <robotNamespace>/billi/default_controller</robotNamespace>
+    <robotSimType>gazebo_ros_control/DefaultRobotHWSim</robotSimType>
+  </plugin>
+</gazebo>
 </robot>
+=======
+</robot>
+>>>>>>> a2351546f9e6cd629167bb84ce18117092a4d7df

File: billi_sim/models/urdf/head.xacro (robot description, xacro)
@@ -3,7 +3,13 @@
    <link name="head">
     <visual>
+<<<<<<< HEAD
+	<origin rpy="3.14 0 1" xyz="0 0 0"/>
+      <geometry>
+        <mesh filename="package://billi_sim/models/meshes/head.stl" scale ="1 1 1"/>
+=======
 	<origin rpy="0 0 0" xyz="0 0 0"/>
       <geometry>
         <mesh filename="package://billi_sim/meshes/head.stl" scale ="1 1 1"/>
+>>>>>>> a2351546f9e6cd629167bb84ce18117092a4d7df
       </geometry>
       <material name="blue"/>
@@ -11,5 +17,9 @@
     <collision>
       <geometry>
+<<<<<<< HEAD
+        <mesh filename="package://billi_sim/models/meshes/head.stl" scale ="1 1 1"/>
+=======
         <mesh filename="package://billi_sim/meshes/head.stl" scale ="1 1 1"/>
+>>>>>>> a2351546f9e6cd629167bb84ce18117092a4d7df
       </geometry>
     </collision>

Commit message: Add files via upload

File: billi_sim/models/urdf/billi.xacro (robot description, xacro)
@@ -2,13 +2,8 @@
 <robot name="billi" xmlns:xacro="http://www.ros.org/wiki/xacro">
   <!-- billi shoulder -->
-<<<<<<< HEAD
 	<!--xacro:include filename="$(find billi_sim)/models/urdf/shoulder.xacro"/-->
-=======
-	<xacro:include filename="$(find billi_sim)/models/urdf/shoulder.xacro"/>
->>>>>>> a2351546f9e6cd629167bb84ce18117092a4d7df
 	<!-- billi body -->
 	<xacro:include filename="$(find billi_sim)/models/urdf/body.xacro"/>
     <!-- billi leg -->
-<<<<<<< HEAD
 	<xacro:include filename="$(find billi_sim)/models/urdf/leg1.xacro"/>
 	<xacro:include filename="$(find billi_sim)/models/urdf/leg2.xacro"/>
@@ -19,21 +14,11 @@
 	<xacro:include filename="$(find billi_sim)/models/urdf/leg-lower1.xacro"/>
 	<xacro:include filename="$(find billi_sim)/models/urdf/leg-lower3.xacro"/>
-=======
-	<xacro:include filename="$(find billi_sim)/models/urdf/leg.xacro"/>
->>>>>>> a2351546f9e6cd629167bb84ce18117092a4d7df
     <!-- billi head -->
 	<xacro:include filename="$(find billi_sim)/models/urdf/head.xacro"/>
-<<<<<<< HEAD
 	<!--gazebo>
 		<plugin name="gazebo_ros_control" filename="libgazebo_ros_control.so"/>
 	</gazebo-->
-=======
-	<gazebo>
-		<plugin name="gazebo_ros_control" filename="libgazebo_ros_control.so"/>
-	</gazebo>
->>>>>>> a2351546f9e6cd629167bb84ce18117092a4d7df
 	<!-- body -->
 	<!-- <xacro:billi_body name="base"/> -->
-<<<<<<< HEAD
 <joint name="lower_upper1" type="revolute">
 			<origin xyz="0.0 -0.039282 0.0" rpy="0 0 0"/>
@@ -90,8 +75,4 @@
     <joint name="head_body" type="revolute">
 			<origin xyz="0.098 0.035 -0.048" rpy="0 0 0"/>
-=======
-    <joint name="head_body" type="revolute">
-			<origin xyz="0 0 0" rpy="0 0 0"/>
->>>>>>> a2351546f9e6cd629167bb84ce18117092a4d7df
 			<parent link="body"/>
 			<child  link="head"/>
@@ -109,9 +90,5 @@
 			<parent link="body"/>
 			<child  link="leg1"/>
-<<<<<<< HEAD
-			<axis xyz="0 0 1"/>
-=======
-			<axis xyz="1 0 0"/>
->>>>>>> a2351546f9e6cd629167bb84ce18117092a4d7df
+			<axis xyz="0 0 1"/>
 			<limit effort="150.0" velocity="12.0"
           lower="-1.57"
@@ -123,35 +100,21 @@
 		</gazebo>
    <joint name="left_hand" type="revolute">
-<<<<<<< HEAD
 			<origin xyz="0 0 -0.092" rpy="0 0 0"/>
 			<parent link="body"/>
 			<child  link="leg4"/>
 			<axis xyz="0 0 1"/>
-=======
-			<origin xyz="0 0 0" rpy="0 0 0"/>
+			<limit effort="150.0" velocity="12.0"
+          lower="-1.57"
+		  upper="1.57"/>
+	</joint>
+<gazebo reference="left_hand">
+		<provideFeedback>true</provideFeedback>
+		<disableFixedJointLumping>true</disableFixedJointLumping>
+		</gazebo>
+ <joint name="right_leg" type="revolute">
+			<origin xyz=".083 .017 0" rpy="0 0 0"/>
 			<parent link="body"/>
 			<child  link="leg2"/>
-			<axis xyz="1 0 0"/>
->>>>>>> a2351546f9e6cd629167bb84ce18117092a4d7df
-			<limit effort="150.0" velocity="12.0"
-          lower="-1.57"
-		  upper="1.57"/>
-	</joint>
-<gazebo reference="left_hand">
-		<provideFeedback>true</provideFeedback>
-		<disableFixedJointLumping>true</disableFixedJointLumping>
-		</gazebo>
- <joint name="right_leg" type="revolute">
-<<<<<<< HEAD
-			<origin xyz=".083 .017 0" rpy="0 0 0"/>
-			<parent link="body"/>
-			<child  link="leg2"/>
-			<axis xyz="0 0 1"/>
-=======
-			<origin xyz="0 0 0" rpy="0 0 0"/>
-			<parent link="body"/>
-			<child  link="leg1"/>
-			<axis xyz="1 0 0"/>
->>>>>>> a2351546f9e6cd629167bb84ce18117092a4d7df
+			<axis xyz="0 0 1"/>
 			<limit effort="150.0" velocity="12.0"
           lower="-1.57"
@@ -163,15 +126,8 @@
 			</gazebo>
     <joint name="left_leg" type="revolute">
-<<<<<<< HEAD
 			<origin xyz="0.083 0.017 -0.092" rpy="0 0 0"/>
 			<parent link="body"/>
 			<child  link="leg3"/>
 			<axis xyz="0 0 1"/>
-=======
-			<origin xyz="0 0 0" rpy="0 0 0"/>
-			<parent link="body"/>
-			<child  link="leg2"/>
-			<axis xyz="1 0 0"/>
->>>>>>> a2351546f9e6cd629167bb84ce18117092a4d7df
 			<limit effort="150.0" velocity="12.0"
           lower="-1.57"
@@ -182,5 +138,4 @@
 		<disableFixedJointLumping>true</disableFixedJointLumping>
 		</gazebo>
-<<<<<<< HEAD
 <!-- Adding transmissions-->
 <transmission name="head">
@@ -281,5 +236,2 @@
 </gazebo>
 </robot>
-=======
-</robot>
->>>>>>> a2351546f9e6cd629167bb84ce18117092a4d7df

File: billi_sim/models/urdf/head.xacro (robot description, xacro)
@@ -3,13 +3,7 @@
    <link name="head">
     <visual>
-<<<<<<< HEAD
 	<origin rpy="3.14 0 1" xyz="0 0 0"/>
       <geometry>
         <mesh filename="package://billi_sim/models/meshes/head.stl" scale ="1 1 1"/>
-=======
-	<origin rpy="0 0 0" xyz="0 0 0"/>
-      <geometry>
-        <mesh filename="package://billi_sim/meshes/head.stl" scale ="1 1 1"/>
->>>>>>> a2351546f9e6cd629167bb84ce18117092a4d7df
       </geometry>
       <material name="blue"/>
@@ -17,9 +11,5 @@
     <collision>
       <geometry>
-<<<<<<< HEAD
         <mesh filename="package://billi_sim/models/meshes/head.stl" scale ="1 1 1"/>
-=======
-        <mesh filename="package://billi_sim/meshes/head.stl" scale ="1 1 1"/>
->>>>>>> a2351546f9e6cd629167bb84ce18117092a4d7df
       </geometry>
     </collision>
