Commit message: champ and billi_sim corrected

File: billi_sim/models/urdf/leg-lower3.xacro (robot description, xacro)
@@ -1,22 +1,26 @@
 <?xml version="1.0"?>
 <robot name="billi" xmlns:xacro="http://www.ros.org/wiki/xacro">
+<!--LEFT LOWER LEG LINK -->
 <link name="leg-lower3">
-    <visual>
-    	<origin rpy="0 3.14 0" xyz="0 0 0"/>
-      <geometry>
-        <mesh filename="package://billi_sim/models/meshes/leg2-lower.stl" scale ="1 1 1"/>
-      </geometry>
-      <material name="blue"/>
-    </visual>
-    <collision>
-      <geometry>
-        <mesh filename="package://billi_sim/models/meshes/leg2-lower.stl" scale ="1 1 1"/>
-      </geometry>
-    </collision>
+    	<visual>
+    		<origin rpy="0 3.14 0" xyz="0 0 0"/>
+      		<geometry>
+        		<mesh filename="package://billi_sim/models/meshes/leg2-lower.stl" scale ="5 5 5"/>
+      		</geometry>
+      		<material name="blue"/>
+    	</visual>
+				<!-- __________________________________ -->
+    	<collision>
+		<origin rpy="0 3.14 0" xyz="0 0 0"/>
+      		<geometry>
+        		<mesh filename="package://billi_sim/models/meshes/leg2-lower.stl" scale ="5 5 5"/>
+     	 	</geometry>
+    	</collision>
+				<!-- __________________________________ -->
 	<inertial>
 		  <mass value="1.0"/>
 		  <origin rpy="0 0 3.14" xyz="0 0 0.1"/>
 		  <inertia ixx="0.0395416666667" ixy="0" ixz="0" iyy="0.106208333333" iyz="0" izz="0.106208333333"/>
-		</inertial>
+	</inertial>
 </link>
 <gazebo reference="leg-lower3">

File: billi_sim/models/urdf/leg-lower4.xacro (robot description, xacro)
@@ -1,22 +1,26 @@
 <?xml version="1.0"?>
 <robot name="billi" xmlns:xacro="http://www.ros.org/wiki/xacro">
+<!--LEFT LOWER HAND LINK -->
 <link name="leg-lower4">
-    <visual>
-    	<origin rpy="0 3.14 0" xyz="0 0 0"/>
-      <geometry>
-        <mesh filename="package://billi_sim/models/meshes/leg2-lower.stl" scale ="1 1 1"/>
-      </geometry>
-      <material name="blue"/>
-    </visual>
-    <collision>
-      <geometry>
-        <mesh filename="package://billi_sim/models/meshes/leg2-lower.stl" scale ="1 1 1"/>
-      </geometry>
-    </collision>
+    	<visual>
+    		<origin rpy="0 3.14 0" xyz="0 0 0"/>
+      		<geometry>
+        		<mesh filename="package://billi_sim/models/meshes/leg2-lower.stl" scale ="5 5 5"/>
+     		</geometry>
+      		<material name="blue"/>
+    	</visual>
+				<!-- __________________________________ -->
+    	<collision>
+		<origin rpy="0 3.14 0" xyz="0 0 0"/>
+      		<geometry>
+        		<mesh filename="package://billi_sim/models/meshes/leg2-lower.stl" scale ="5 5 5"/>
+      		</geometry>
+    	</collision>
+				<!-- __________________________________ -->
 	<inertial>
 		  <mass value="1.0"/>
 		  <origin rpy="0 0 3.14" xyz="0 0 0.1"/>
 		  <inertia ixx="0.0395416666667" ixy="0" ixz="0" iyy="0.106208333333" iyz="0" izz="0.106208333333"/>
-		</inertial>
+	</inertial>
 </link>
 <gazebo reference="leg-lower4">

File: billi_sim/models/urdf/leg1.xacro (robot description, xacro)
@@ -1,22 +1,26 @@
 <?xml version="1.0"?>
 <robot name="billi" xmlns:xacro="http://www.ros.org/wiki/xacro">
+<!--RIGHT HAND LINK -->
 <link name="leg1">
-    <visual>
-    	<origin rpy="0 0 0" xyz="0 0 0"/>
-      <geometry>
-        <mesh filename="package://billi_sim/models/meshes/leg-upper.stl" scale ="1 1 1"/>
-      </geometry>
-      <material name="blue"/>
-    </visual>
-    <collision>
-      <geometry>
-        <mesh filename="package://billi_sim/models/meshes/leg-upper.stl" scale ="1 1 1"/>
-      </geometry>
-    </collision>
+    	<visual>
+    		<origin rpy="0 0 0" xyz="0 0 0"/>
+     	 	<geometry>
+        		<mesh filename="package://billi_sim/models/meshes/leg-upper.stl" scale ="5 5 5"/>
+      		</geometry>
+      		<material name="blue"/>
+    	</visual>
+				<!-- __________________________________ -->
+   	<collision>
+		<origin rpy="0 0 0" xyz="0 0 0"/>
+      		<geometry>
+        		<mesh filename="package://billi_sim/models/meshes/leg-upper.stl" scale ="5 5 5"/>
+      		</geometry>
+    	</collision>
+				<!-- __________________________________ -->
 	<inertial>
 		  <mass value="1.0"/>
 		  <origin rpy="0 0 0" xyz="0 0 0.1"/>
-		  <inertia ixx="0.0395416666667" ixy="0" ixz="0" iyy="0.106208333333" iyz="0" izz="0.106208333333"/>
-		</inertial>
+		  <inertia ixx="0.13157" ixy="0" ixz="0" iyy="0.01122" iyz="0" izz="0.14025"/>
+	</inertial>
 </link>
 <gazebo reference="leg1">

File: billi_sim/models/urdf/leg2.xacro (robot description, xacro)
@@ -1,23 +1,27 @@
 <?xml version="1.0"?>
 <robot name="billi" xmlns:xacro="http://www.ros.org/wiki/xacro">
+<!--RIGHT LEG LINK -->
 <link name="leg2">
-    <visual>
-	<origin rpy="0 0 0" xyz="0 0 0"/>
-      <geometry>
-        <mesh filename="package://billi_sim/models/meshes/leg-upper.stl" scale ="1 1 1"/>
-      </geometry>
-      <material name="blue"/>
-    </visual>
-    <collision>
-      <geometry>
-        <mesh filename="package://billi_sim/models/meshes/leg-upper.stl" scale ="1 1 1"/>
-      </geometry>
-    </collision>
+    	<visual>
+		<origin rpy="0 0 0" xyz="0 0 0"/>
+      		<geometry>
+        		<mesh filename="package://billi_sim/models/meshes/leg-upper.stl" scale ="5 5 5"/>
+     	 	</geometry>
+      		<material name="blue"/>
+    	</visual>
+				<!-- __________________________________ -->
+    	<collision>
+		<origin rpy="0 0 0" xyz="0 0 0"/>
+      		<geometry>
+        		<mesh filename="package://billi_sim/models/meshes/leg-upper.stl" scale ="5 5 5"/>
+      		</geometry>
+    	</collision>
+				<!-- __________________________________ -->
 	<inertial>
 		  <mass value="1.0"/>
 		  <origin rpy="0 0 0" xyz="0 0 0.1"/>
-		  <inertia ixx="0.0395416666667" ixy="0" ixz="0" iyy="0.106208333333" iyz="0" izz="0.106208333333"/>
-		</inertial>
-   </link>
+		  <inertia ixx="0.13157" ixy="0" ixz="0" iyy="0.01122" iyz="0" izz="0.14025"/>
+	</inertial>
+</link>
 <gazebo reference="leg2">
         <kp>1000.0</kp>

File: billi_sim/models/urdf/leg3.xacro (robot description, xacro)
@@ -1,23 +1,27 @@
 <?xml version="1.0"?>
 <robot name="billi" xmlns:xacro="http://www.ros.org/wiki/xacro">
+<!--LEFT LEG LINK -->
 <link name="leg3">
-    <visual>
-	<origin rpy="0 3.14 0" xyz="0 0 0"/>
-      <geometry>
-        <mesh filename="package://billi_sim/models/meshes/leg-upper.stl" scale ="1 1 1"/>
-      </geometry>
-      <material name="blue"/>
-    </visual>
-    <collision>
-      <geometry>
-        <mesh filename="package://billi_sim/models/meshes/leg-upper.stl" scale ="1 1 1"/>
-      </geometry>
-    </collision>
+    	<visual>
+		<origin rpy="0 3.14 0" xyz="0 0 0"/>
+     		<geometry>
+       			<mesh filename="package://billi_sim/models/meshes/leg-upper.stl" scale ="5 5 5"/>
+      		</geometry>
+     		<material name="blue"/>
+    	</visual>
+				<!-- __________________________________ -->
+    	<collision>
+		<origin rpy="0 3.14 0" xyz="0 0 0"/>
+      		<geometry>
+        		<mesh filename="package://billi_sim/models/meshes/leg-upper.stl" scale ="5 5 5"/>
+      		</geometry>
+    	</collision>
+				<!-- __________________________________ -->
 	<inertial>
 		  <mass value="1.0"/>
 		  <origin rpy="0 0 0" xyz="0 0 0.1"/>
-		  <inertia ixx="0.0395416666667" ixy="0" ixz="0" iyy="0.106208333333" iyz="0" izz="0.106208333333"/>
-		</inertial>
-   </link>
+		  <inertia ixx="0.13157" ixy="0" ixz="0" iyy="0.01122" iyz="0" izz="0.14025"/>
+	</inertial>
+</link>
 <gazebo reference="leg3">
         <kp>1000.0</kp>

File: billi_sim/models/urdf/leg4.xacro (robot description, xacro)
@@ -1,23 +1,27 @@
 <?xml version="1.0"?>
 <robot name="billi" xmlns:xacro="http://www.ros.org/wiki/xacro">
+<!--LEFT HAND LINK -->
 <link name="leg4">
-    <visual>
-	<origin rpy="0 3.14 0" xyz="0 0 0"/>
-      <geometry>
-        <mesh filename="package://billi_sim/models/meshes/leg-upper.stl" scale ="1 1 1"/>
-      </geometry>
-      <material name="blue"/>
-    </visual>
-    <collision>
-      <geometry>
-        <mesh filename="package://billi_sim/models/meshes/leg-upper.stl" scale ="1 1 1"/>
-      </geometry>
-    </collision>
+    	<visual>
+		<origin rpy="0 3.14 0" xyz="0 0 0"/>
+      		<geometry>
+        		<mesh filename="package://billi_sim/models/meshes/leg-upper.stl" scale ="5 5 5"/>
+      		</geometry>
+      		<material name="blue"/>
+    	</visual>
+				<!-- __________________________________ -->
+    	<collision>
+		<origin rpy="0 3.14 0" xyz="0 0 0"/>
+      		<geometry>
+        		<mesh filename="package://billi_sim/models/meshes/leg-upper.stl" scale ="5 5 5"/>
+      		</geometry>
+    	</collision>
+				<!-- __________________________________ -->
 	<inertial>
 		  <mass value="1.0"/>
 		  <origin rpy="0 0 0" xyz="0 0 0.1"/>
-		  <inertia ixx="0.0395416666667" ixy="0" ixz="0" iyy="0.106208333333" iyz="0" izz="0.106208333333"/>
-		</inertial>
-   </link>
+		  <inertia ixx="0.13157" ixy="0" ixz="0" iyy="0.01122" iyz="0" izz="0.14025"/>
+	</inertial>
+</link>
 <gazebo reference="leg4">
         <kp>1000.0</kp>
