Commit message: Fix link tree disconnect

File: champ/champ_description/urdf/accessories.urdf.xacro (robot description, xacro)
@@ -16,9 +16,9 @@
 		<material>Gazebo/FlatBlack</material>
 	</gazebo>
-    <xacro:asus_camera
+    <!-- <xacro:asus_camera
         parent="base_link"
         name="camera">
         <origin xyz="${base_x_length / 2} 0.0 ${base_z_length / 2 + 0.01}" rpy="0 0 0"/>
-    </xacro:asus_camera>
+    </xacro:asus_camera> -->
     <gazebo>
         <plugin name="imu_controller" filename="libhector_gazebo_ros_imu.so">

File: champ/champ_description/urdf/champ.urdf (robot description, URDF)
Before this commit: robot champ, 25 links, 24 joints
Links:
- added link camera_depth_frame
- added link camera_depth_optical_frame
- added link camera_rgb_frame
- added link camera_rgb_optical_frame
- added link stereo_cam_link, mass 0.001
Joints:
- added joint camera_depth_joint: type fixed, parent camera_link, child camera_depth_frame, origin xyz=0.0 0.049 0.0 rpy=0 0 0
- added joint camera_depth_optical_joint: type fixed, parent camera_depth_frame, child camera_depth_optical_frame, origin xyz=0 0 0 rpy=-1.57079632679 0.0 -1.57079632679
- added joint camera_rgb_joint: type fixed, parent camera_link, child camera_rgb_frame, origin xyz=0.0 0.022 0.0 rpy=0 0 0
- added joint camera_rgb_optical_joint: type fixed, parent camera_rgb_frame, child camera_rgb_optical_frame, origin xyz=0 0 0 rpy=-1.57079632679 0.0 -1.57079632679
- added joint stereo_cam_joint: type fixed, parent base_link, child stereo_cam_link

Commit message: stereo camera added

File: champ/champ_description/urdf/accessories.urdf.xacro (robot description, xacro)
@@ -21,4 +21,34 @@
         <origin xyz="${base_x_length / 2} 0.0 ${base_z_length / 2 + 0.01}" rpy="0 0 0"/>
     </xacro:asus_camera> -->
+  <link name="stereo_cam_link">
+    <inertial>
+      <mass value="0.001"/>
+      <origin xyz="0 0 0" rpy="0 0 0"/>
+      <inertia ixx="1e-09" ixy="0.0" ixz="0.0" iyy="1e-09" iyz="0.0" izz="1e-09"/>
+    </inertial>
+  </link>
+  <joint name="stereo_cam_joint" type="fixed">
+    <parent link="base_link" />
+    <child link="stereo_cam_link" />
+  </joint>
+    <gazebo>
+      <sensor>
+        <plugin filename="libgazebo_ros_multicamera.so" name="stereo_camera_controller">
+        <alwaysOn>true</alwaysOn>
+        <updateRate>0.0</updateRate>
+        <cameraName>billi/camera</cameraName>
+        <imageTopicName>image_raw</imageTopicName>
+        <cameraInfoTopicName>/camera_info</cameraInfoTopicName>
+        <frameName>left_camera_frame</frameName>
+        <!-- <rightFrameName>right_camera_frame</rightFrameName> -->
+        <hackBaseline>0.07</hackBaseline>
+        <distortionK1>0.0</distortionK1>
+        <distortionK2>0.0</distortionK2>
+        <distortionK3>0.0</distortionK3>
+        <distortionT1>0.0</distortionT1>
+        <distortionT2>0.0</distortionT2>
+      </plugin>
+     </sensor>
+    </gazebo>
     <gazebo>
         <plugin name="imu_controller" filename="libhector_gazebo_ros_imu.so">

File: champ/champ_description/urdf/champ.urdf (robot description, URDF)
Before this commit: robot champ, 30 links, 29 joints
Links:
- removed link camera_depth_frame
- removed link camera_depth_optical_frame
- removed link camera_rgb_frame
- removed link camera_rgb_optical_frame
Joints:
- removed joint camera_depth_joint
- removed joint camera_depth_optical_joint
- removed joint camera_rgb_joint
- removed joint camera_rgb_optical_joint

File: champ/champ_description/urdf/champ.urdf.xacro (robot description, xacro)
@@ -41,4 +41,34 @@
     <xacro:champ_leg leg="rf"/>
     <xacro:champ_leg leg="rh"/>
+  <link name="stereo_cam_link">
+    <inertial>
+      <mass value="0.001"/>
+      <origin xyz="0 0 0" rpy="0 0 0"/>
+      <inertia ixx="1e-09" ixy="0.0" ixz="0.0" iyy="1e-09" iyz="0.0" izz="1e-09"/>
+    </inertial>
+  </link>
+  <joint name="stereo_cam_joint" type="fixed">
+    <parent link="base_link" />
+    <child link="stereo_cam_link" />
+  </joint>
+    <gazebo>
+      <sensor>
+        <plugin filename="libgazebo_ros_multicamera.so" name="stereo_camera_controller">
+        <alwaysOn>true</alwaysOn>
+        <updateRate>0.0</updateRate>
+        <cameraName>billi/camera</cameraName>
+        <imageTopicName>image_raw</imageTopicName>
+        <cameraInfoTopicName>/camera_info</cameraInfoTopicName>
+        <frameName>left_camera_frame</frameName>
+        <!-- <rightFrameName>right_camera_frame</rightFrameName> -->
+        <hackBaseline>0.07</hackBaseline>
+        <distortionK1>0.0</distortionK1>
+        <distortionK2>0.0</distortionK2>
+        <distortionK3>0.0</distortionK3>
+        <distortionT1>0.0</distortionT1>
+        <distortionT2>0.0</distortionT2>
+      </plugin>
+     </sensor>
+    </gazebo>
     <gazebo>
       <plugin name="p3d_base_controller" filename="libgazebo_ros_p3d.so">

Commit message: stereo camera added

File: champ/champ_description/urdf/accessories.urdf.xacro (robot description, xacro)
@@ -3,5 +3,4 @@
     <xacro:include filename="$(find hector_sensors_description)/urdf/hokuyo_utm30lx.urdf.xacro" />
     <xacro:include filename="$(find hector_sensors_description)/urdf/asus_camera.urdf.xacro" />
-<<<<<<< HEAD
     <xacro:hokuyo_utm30lx
         name="hokuyo"
@@ -14,26 +13,7 @@
         <origin xyz="0.0 0.0 ${base_z_length / 2 + 0.04}" rpy="0 0 0"/>
     </xacro:hokuyo_utm30lx>
-=======
-    <xacro:hokuyo_utm30lx
-        name="hokuyo"
-        parent="base_link"
-        ros_topic="scan"
-        update_rate="30"
-        ray_count="1040"
-        min_angle="130"
-        max_angle="-130" >
-        <origin xyz="0.0 0.0 ${base_z_length / 2 + 0.04}" rpy="0 0 0"/>
-    </xacro:hokuyo_utm30lx>
->>>>>>> champ
     <gazebo reference="hokuyo_frame">
 		<material>Gazebo/FlatBlack</material>
 	</gazebo>
-<<<<<<< HEAD
-    <xacro:asus_camera_model
-        parent="base_link"
-        name="camera">
-        <origin xyz="${base_x_length / 2} 0.0 ${base_z_length / 2 + 0.01}" rpy="0 0 0"/>
-    </xacro:asus_camera_model>
-=======
     <!-- <xacro:asus_camera
         parent="base_link"
@@ -71,5 +51,4 @@
      </sensor>
     </gazebo>
->>>>>>> champ
     <gazebo>
         <plugin name="imu_controller" filename="libhector_gazebo_ros_imu.so">
@@ -100,6 +79,3 @@
         <origin xyz="0.07 0.0 ${base_z_length / 2}" rpy="0 0 0"/>
     </xacro:champ_arm> -->
-<<<<<<< HEAD
-=======
->>>>>>> champ
 </robot>

File: champ/champ_description/urdf/champ.urdf.xacro (robot description, xacro)
@@ -41,6 +41,4 @@
     <xacro:champ_leg leg="rf"/>
     <xacro:champ_leg leg="rh"/>
-<<<<<<< HEAD
-=======
   <link name="stereo_cam_link">
     <inertial>
@@ -73,5 +71,4 @@
      </sensor>
     </gazebo>
->>>>>>> champ
     <gazebo>
       <plugin name="p3d_base_controller" filename="libgazebo_ros_p3d.so">

Commit message: Revert "Stereo_cam Added in champModel"

File: champ/champ_description/urdf/accessories.urdf.xacro (robot description, xacro)
@@ -16,39 +16,9 @@
 		<material>Gazebo/FlatBlack</material>
 	</gazebo>
-    <!-- <xacro:asus_camera
+    <xacro:asus_camera_model
         parent="base_link"
         name="camera">
         <origin xyz="${base_x_length / 2} 0.0 ${base_z_length / 2 + 0.01}" rpy="0 0 0"/>
-    </xacro:asus_camera> -->
-  <link name="stereo_cam_link">
-    <inertial>
-      <mass value="0.001"/>
-      <origin xyz="0 0 0" rpy="0 0 0"/>
-      <inertia ixx="1e-09" ixy="0.0" ixz="0.0" iyy="1e-09" iyz="0.0" izz="1e-09"/>
-    </inertial>
-  </link>
-  <joint name="stereo_cam_joint" type="fixed">
-    <parent link="base_link" />
-    <child link="stereo_cam_link" />
-  </joint>
-    <gazebo>
-      <sensor>
-        <plugin filename="libgazebo_ros_multicamera.so" name="stereo_camera_controller">
-        <alwaysOn>true</alwaysOn>
-        <updateRate>0.0</updateRate>
-        <cameraName>billi/camera</cameraName>
-        <imageTopicName>image_raw</imageTopicName>
-        <cameraInfoTopicName>/camera_info</cameraInfoTopicName>
-        <frameName>left_camera_frame</frameName>
-        <!-- <rightFrameName>right_camera_frame</rightFrameName> -->
-        <hackBaseline>0.07</hackBaseline>
-        <distortionK1>0.0</distortionK1>
-        <distortionK2>0.0</distortionK2>
-        <distortionK3>0.0</distortionK3>
-        <distortionT1>0.0</distortionT1>
-        <distortionT2>0.0</distortionT2>
-      </plugin>
-     </sensor>
-    </gazebo>
+    </xacro:asus_camera_model>
     <gazebo>
         <plugin name="imu_controller" filename="libhector_gazebo_ros_imu.so">

File: champ/champ_description/urdf/champ.urdf (robot description, URDF)
Before this commit: robot champ, 26 links, 25 joints
Links:
- removed link lf_hip_debug_link
- removed link lf_hip_link
- removed link lh_hip_debug_link
- removed link lh_hip_link
- removed link rf_hip_debug_link
- removed link rf_hip_link
- removed link rh_hip_debug_link
- removed link rh_hip_link
- removed link stereo_cam_link
- added link camera_depth_frame
- added link camera_depth_optical_frame
- added link camera_rgb_frame
- added link camera_rgb_optical_frame
- link base_link: geometry collision mesh filename=package://champ_description/meshes/base.stl scale=1 1 1; visual mesh filename=package://champ_description/meshes/base.stl scale=1 1 1
- link lf_lower_leg_link: geometry collision mesh filename=package://champ_description/meshes/lower_leg3.stl scale=1 1 1; visual mesh filename=package://champ_description/meshes/lower_leg3.stl scale=1 1 1
- link lf_upper_leg_link: geometry collision mesh filename=package://champ_description/meshes/upper_leg3.stl scale=1 1 1; visual mesh filename=package://champ_description/meshes/upper_leg3.stl scale=1 1 1
- link lh_lower_leg_link: geometry collision mesh filename=package://champ_description/meshes/lower_leg4.stl scale=0.001 0.001 0.001; visual mesh filename=package://champ_description/meshes/lower_leg4.stl scale=0.001 0.001 0.001
- link lh_upper_leg_link: geometry collision mesh filename=package://champ_description/meshes/upper_leg4.stl scale=0.001 0.001 0.001; visual mesh filename=package://champ_description/meshes/upper_leg4.stl scale=0.001 0.001 0.001
- link rf_lower_leg_link: geometry collision mesh filename=package://champ_description/meshes/lower_leg2.stl scale=0.001 0.001 0.001; visual mesh filename=package://champ_description/meshes/lower_leg2.stl scale=0.001 0.001 0.001
- link rf_upper_leg_link: geometry collision mesh filename=package://champ_description/meshes/upper_leg2.stl scale=0.001 0.001 0.001; visual mesh filename=package://champ_description/meshes/upper_leg2.stl scale=0.001 0.001 0.001
- link rh_lower_leg_link: geometry collision mesh filename=package://champ_description/meshes/lower_leg1.stl scale=0.001 0.001 0.001; visual mesh filename=package://champ_description/meshes/lower_leg1.stl scale=0.001 0.001 0.001
- link rh_upper_leg_link: geometry collision mesh filename=package://champ_description/meshes/upper_leg1.stl scale=0.001 0.001 0.001; visual mesh filename=package://champ_description/meshes/upper_leg1.stl scale=0.001 0.001 0.001
Joints:
- removed joint lf_debug_joint
- removed joint lf_hip_joint
- removed joint lh_debug_joint
- removed joint lh_hip_joint
- removed joint rf_debug_joint
- removed joint rf_hip_joint
- removed joint rh_debug_joint
- removed joint rh_hip_joint
- removed joint stereo_cam_joint
- added joint camera_depth_joint: type fixed, parent camera_link, child camera_depth_frame, origin xyz=0.0 0.049 0.0 rpy=0 0 0
- added joint camera_depth_optical_joint: type fixed, parent camera_depth_frame, child camera_depth_optical_frame, origin xyz=0 0 0 rpy=-1.57079632679 0.0 -1.57079632679
- added joint camera_rgb_joint: type fixed, parent camera_link, child camera_rgb_frame, origin xyz=0.0 0.022 0.0 rpy=0 0 0
- added joint camera_rgb_optical_joint: type fixed, parent camera_rgb_frame, child camera_rgb_optical_frame, origin xyz=0 0 0 rpy=-1.57079632679 0.0 -1.57079632679
- joint lf_lower_leg_joint: axis 0 1 0 -> 0 0 1; limit lower=-3.14159265359 upper=3.14159265359 effort=25 velocity=1.5 -> lower=-3.14159265359 upper=3.14159265359 effort=25 velocity=0.1; origin xyz=0 0 -0.141 rpy=0 0 0 -> xyz=0.0 -0.039282 0.0 rpy=0 0 0
- joint lf_upper_leg_joint: axis 0 1 0 -> 0 0 1; limit lower=-3.14159265359 upper=3.14159265359 effort=25 velocity=1.5 -> lower=-3.14159265359 upper=3.14159265359 effort=25 velocity=0.1; origin xyz=0 0.06 0 rpy=0 0 0 -> xyz=0.083 0.017 -0.092 rpy=0 0 0; parent lf_hip_link -> base_link
- joint lh_lower_leg_joint: axis 0 1 0 -> 0 0 1; limit lower=-3.14159265359 upper=3.14159265359 effort=25 velocity=1.5 -> lower=-3.14159265359 upper=3.14159265359 effort=25 velocity=0.1; origin xyz=0 0 -0.141 rpy=0 0 0 -> xyz=0.0 -0.039282 0.0 rpy=0 0 0
- joint lh_upper_leg_joint: axis 0 1 0 -> 0 0 1; limit lower=-3.14159265359 upper=3.14159265359 effort=25 velocity=1.5 -> lower=-3.14159265359 upper=3.14159265359 effort=25 velocity=0.1; origin xyz=0 0.06 0 rpy=0 0 0 -> xyz=0 0 -0.092 rpy=0 0 0; parent lh_hip_link -> base_link
- joint rf_lower_leg_joint: axis 0 1 0 -> 0 0 1; limit lower=-3.14159265359 upper=3.14159265359 effort=25 velocity=1.5 -> lower=-3.14159265359 upper=3.14159265359 effort=25 velocity=0.1; origin xyz=0 0 -0.141 rpy=0 0 0 -> xyz=0.0 -0.039282 0.0 rpy=0 0 0
- joint rf_upper_leg_joint: axis 0 1 0 -> 0 0 1; limit lower=-3.14159265359 upper=3.14159265359 effort=25 velocity=1.5 -> lower=-3.14159265359 upper=3.14159265359 effort=25 velocity=0.1; origin xyz=0 -0.06 0 rpy=0 0 0 -> xyz=.083 .017 0 rpy=0 0 0; parent rf_hip_link -> base_link
- joint rh_lower_leg_joint: axis 0 1 0 -> 0 0 1; limit lower=-3.14159265359 upper=3.14159265359 effort=25 velocity=1.5 -> lower=-3.14159265359 upper=3.14159265359 effort=25 velocity=0.1; origin xyz=0 0 -0.141 rpy=0 0 0 -> xyz=0.0 -0.039282 0.0 rpy=0 0 0
- joint rh_upper_leg_joint: axis 0 1 0 -> 0 0 1; limit lower=-3.14159265359 upper=3.14159265359 effort=25 velocity=1.5 -> lower=-3.14159265359 upper=3.14159265359 effort=25 velocity=0.1; origin xyz=0 -0.06 0 rpy=0 0 0 -> xyz=0 0 0 rpy=0 0 0; parent rh_hip_link -> base_link

File: champ/champ_description/urdf/champ.urdf.xacro (robot description, xacro)
@@ -41,34 +41,4 @@
     <xacro:champ_leg leg="rf"/>
     <xacro:champ_leg leg="rh"/>
-  <link name="stereo_cam_link">
-    <inertial>
-      <mass value="0.001"/>
-      <origin xyz="0 0 0" rpy="0 0 0"/>
-      <inertia ixx="1e-09" ixy="0.0" ixz="0.0" iyy="1e-09" iyz="0.0" izz="1e-09"/>
-    </inertial>
-  </link>
-  <joint name="stereo_cam_joint" type="fixed">
-    <parent link="base_link" />
-    <child link="stereo_cam_link" />
-  </joint>
-    <gazebo>
-      <sensor>
-        <plugin filename="libgazebo_ros_multicamera.so" name="stereo_camera_controller">
-        <alwaysOn>true</alwaysOn>
-        <updateRate>0.0</updateRate>
-        <cameraName>billi/camera</cameraName>
-        <imageTopicName>image_raw</imageTopicName>
-        <cameraInfoTopicName>/camera_info</cameraInfoTopicName>
-        <frameName>left_camera_frame</frameName>
-        <!-- <rightFrameName>right_camera_frame</rightFrameName> -->
-        <hackBaseline>0.07</hackBaseline>
-        <distortionK1>0.0</distortionK1>
-        <distortionK2>0.0</distortionK2>
-        <distortionK3>0.0</distortionK3>
-        <distortionT1>0.0</distortionT1>
-        <distortionT2>0.0</distortionT2>
-      </plugin>
-     </sensor>
-    </gazebo>
     <gazebo>
       <plugin name="p3d_base_controller" filename="libgazebo_ros_p3d.so">

Commit message: upstream pulled and stereo camera added

File: champ/champ_description/urdf/accessories.urdf.xacro (robot description, xacro)
@@ -16,9 +16,9 @@
 		<material>Gazebo/FlatBlack</material>
 	</gazebo>
-    <!-- <xacro:asus_camera
+    <!--<xacro:asus_camera_model
         parent="base_link"
         name="camera">
         <origin xyz="${base_x_length / 2} 0.0 ${base_z_length / 2 + 0.01}" rpy="0 0 0"/>
-    </xacro:asus_camera> -->
+    </xacro:asus_camera_model>-->
   <link name="stereo_cam_link">
     <inertial>

File: champ/champ_description/urdf/champ.urdf (robot description, URDF)
Before this commit: robot champ, 26 links, 25 joints
Links:
- removed link lf_hip_debug_link
- removed link lf_hip_link
- removed link lh_hip_debug_link
- removed link lh_hip_link
- removed link rf_hip_debug_link
- removed link rf_hip_link
- removed link rh_hip_debug_link
- removed link rh_hip_link
- link base_link: geometry collision mesh filename=package://champ_description/meshes/base.stl scale=1 1 1; visual mesh filename=package://champ_description/meshes/base.stl scale=1 1 1
- link lf_lower_leg_link: geometry collision mesh filename=package://champ_description/meshes/lower_leg3.stl scale=1 1 1; visual mesh filename=package://champ_description/meshes/lower_leg3.stl scale=1 1 1
- link lf_upper_leg_link: geometry collision mesh filename=package://champ_description/meshes/upper_leg3.stl scale=1 1 1; visual mesh filename=package://champ_description/meshes/upper_leg3.stl scale=1 1 1
- link lh_lower_leg_link: geometry collision mesh filename=package://champ_description/meshes/lower_leg4.stl scale=0.001 0.001 0.001; visual mesh filename=package://champ_description/meshes/lower_leg4.stl scale=0.001 0.001 0.001
- link lh_upper_leg_link: geometry collision mesh filename=package://champ_description/meshes/upper_leg4.stl scale=0.001 0.001 0.001; visual mesh filename=package://champ_description/meshes/upper_leg4.stl scale=0.001 0.001 0.001
- link rf_lower_leg_link: geometry collision mesh filename=package://champ_description/meshes/lower_leg2.stl scale=0.001 0.001 0.001; visual mesh filename=package://champ_description/meshes/lower_leg2.stl scale=0.001 0.001 0.001
- link rf_upper_leg_link: geometry collision mesh filename=package://champ_description/meshes/upper_leg2.stl scale=0.001 0.001 0.001; visual mesh filename=package://champ_description/meshes/upper_leg2.stl scale=0.001 0.001 0.001
- link rh_lower_leg_link: geometry collision mesh filename=package://champ_description/meshes/lower_leg1.stl scale=0.001 0.001 0.001; visual mesh filename=package://champ_description/meshes/lower_leg1.stl scale=0.001 0.001 0.001
- link rh_upper_leg_link: geometry collision mesh filename=package://champ_description/meshes/upper_leg1.stl scale=0.001 0.001 0.001; visual mesh filename=package://champ_description/meshes/upper_leg1.stl scale=0.001 0.001 0.001
Joints:
- removed joint lf_debug_joint
- removed joint lf_hip_joint
- removed joint lh_debug_joint
- removed joint lh_hip_joint
- removed joint rf_debug_joint
- removed joint rf_hip_joint
- removed joint rh_debug_joint
- removed joint rh_hip_joint
- joint lf_lower_leg_joint: axis 0 1 0 -> 0 0 1; limit lower=-3.14159265359 upper=3.14159265359 effort=25 velocity=1.5 -> lower=-3.14159265359 upper=3.14159265359 effort=25 velocity=0.1; origin xyz=0 0 -0.141 rpy=0 0 0 -> xyz=0.0 -0.039282 0.0 rpy=0 0 0
- joint lf_upper_leg_joint: axis 0 1 0 -> 0 0 1; limit lower=-3.14159265359 upper=3.14159265359 effort=25 velocity=1.5 -> lower=-3.14159265359 upper=3.14159265359 effort=25 velocity=0.1; origin xyz=0 0.06 0 rpy=0 0 0 -> xyz=0.083 0.017 -0.092 rpy=0 0 0; parent lf_hip_link -> base_link
- joint lh_lower_leg_joint: axis 0 1 0 -> 0 0 1; limit lower=-3.14159265359 upper=3.14159265359 effort=25 velocity=1.5 -> lower=-3.14159265359 upper=3.14159265359 effort=25 velocity=0.1; origin xyz=0 0 -0.141 rpy=0 0 0 -> xyz=0.0 -0.039282 0.0 rpy=0 0 0
- joint lh_upper_leg_joint: axis 0 1 0 -> 0 0 1; limit lower=-3.14159265359 upper=3.14159265359 effort=25 velocity=1.5 -> lower=-3.14159265359 upper=3.14159265359 effort=25 velocity=0.1; origin xyz=0 0.06 0 rpy=0 0 0 -> xyz=0 0 -0.092 rpy=0 0 0; parent lh_hip_link -> base_link
- joint rf_lower_leg_joint: axis 0 1 0 -> 0 0 1; limit lower=-3.14159265359 upper=3.14159265359 effort=25 velocity=1.5 -> lower=-3.14159265359 upper=3.14159265359 effort=25 velocity=0.1; origin xyz=0 0 -0.141 rpy=0 0 0 -> xyz=0.0 -0.039282 0.0 rpy=0 0 0
- joint rf_upper_leg_joint: axis 0 1 0 -> 0 0 1; limit lower=-3.14159265359 upper=3.14159265359 effort=25 velocity=1.5 -> lower=-3.14159265359 upper=3.14159265359 effort=25 velocity=0.1; origin xyz=0 -0.06 0 rpy=0 0 0 -> xyz=.083 .017 0 rpy=0 0 0; parent rf_hip_link -> base_link
- joint rh_lower_leg_joint: axis 0 1 0 -> 0 0 1; limit lower=-3.14159265359 upper=3.14159265359 effort=25 velocity=1.5 -> lower=-3.14159265359 upper=3.14159265359 effort=25 velocity=0.1; origin xyz=0 0 -0.141 rpy=0 0 0 -> xyz=0.0 -0.039282 0.0 rpy=0 0 0
- joint rh_upper_leg_joint: axis 0 1 0 -> 0 0 1; limit lower=-3.14159265359 upper=3.14159265359 effort=25 velocity=1.5 -> lower=-3.14159265359 upper=3.14159265359 effort=25 velocity=0.1; origin xyz=0 -0.06 0 rpy=0 0 0 -> xyz=0 0 0 rpy=0 0 0; parent rh_hip_link -> base_link
