Commit message: upstream pulled and stereo camera added

File: champ/champ_description/urdf/accessories.urdf.xacro (robot description, xacro)
@@ -16,9 +16,9 @@
 		<material>Gazebo/FlatBlack</material>
 	</gazebo>
-    <!--<xacro:asus_camera_model
+    <!-- <xacro:asus_camera
         parent="base_link"
         name="camera">
         <origin xyz="${base_x_length / 2} 0.0 ${base_z_length / 2 + 0.01}" rpy="0 0 0"/>
-    </xacro:asus_camera_model>-->
+    </xacro:asus_camera> -->
   <link name="stereo_cam_link">
     <inertial>

File: champ/champ_description/urdf/champ.urdf (robot description, URDF)
Before this commit: robot champ, 18 links, 17 joints
Links:
- added link lf_hip_debug_link
- added link lf_hip_link, mass 0.25; collision mesh filename=package://champ_description/meshes/hip.stl scale=0.001 0.001 0.001; visual mesh filename=package://champ_description/meshes/hip.stl scale=0.001 0.001 0.001
- added link lh_hip_debug_link
- added link lh_hip_link, mass 0.25; collision mesh filename=package://champ_description/meshes/hip.stl scale=0.001 0.001 0.001; visual mesh filename=package://champ_description/meshes/hip.stl scale=0.001 0.001 0.001
- added link rf_hip_debug_link
- added link rf_hip_link, mass 0.25; collision mesh filename=package://champ_description/meshes/hip.stl scale=0.001 0.001 0.001; visual mesh filename=package://champ_description/meshes/hip.stl scale=0.001 0.001 0.001
- added link rh_hip_debug_link
- added link rh_hip_link, mass 0.25; collision mesh filename=package://champ_description/meshes/hip.stl scale=0.001 0.001 0.001; visual mesh filename=package://champ_description/meshes/hip.stl scale=0.001 0.001 0.001
- link base_link: geometry collision mesh filename=package://champ_description/meshes/base.stl scale=0.001 0.001 0.001; visual mesh filename=package://champ_description/meshes/base.stl scale=0.001 0.001 0.001
- link lf_lower_leg_link: geometry collision mesh filename=package://champ_description/meshes/lower_leg.stl scale=0.001 0.001 0.001; visual mesh filename=package://champ_description/meshes/lower_leg.stl scale=0.001 0.001 0.001
- link lf_upper_leg_link: geometry collision mesh filename=package://champ_description/meshes/upper_leg.stl scale=0.001 0.001 0.001; visual mesh filename=package://champ_description/meshes/upper_leg.stl scale=0.001 0.001 0.001
- link lh_lower_leg_link: geometry collision mesh filename=package://champ_description/meshes/lower_leg.stl scale=0.001 0.001 0.001; visual mesh filename=package://champ_description/meshes/lower_leg.stl scale=0.001 0.001 0.001
- link lh_upper_leg_link: geometry collision mesh filename=package://champ_description/meshes/upper_leg.stl scale=0.001 0.001 0.001; visual mesh filename=package://champ_description/meshes/upper_leg.stl scale=0.001 0.001 0.001
- link rf_lower_leg_link: geometry collision mesh filename=package://champ_description/meshes/lower_leg.stl scale=0.001 0.001 0.001; visual mesh filename=package://champ_description/meshes/lower_leg.stl scale=0.001 0.001 0.001
- link rf_upper_leg_link: geometry collision mesh filename=package://champ_description/meshes/upper_leg.stl scale=0.001 0.001 0.001; visual mesh filename=package://champ_description/meshes/upper_leg.stl scale=0.001 0.001 0.001
- link rh_lower_leg_link: geometry collision mesh filename=package://champ_description/meshes/lower_leg.stl scale=0.001 0.001 0.001; visual mesh filename=package://champ_description/meshes/lower_leg.stl scale=0.001 0.001 0.001
- link rh_upper_leg_link: geometry collision mesh filename=package://champ_description/meshes/upper_leg.stl scale=0.001 0.001 0.001; visual mesh filename=package://champ_description/meshes/upper_leg.stl scale=0.001 0.001 0.001
Joints:
- added joint lf_debug_joint: type fixed, parent base_link, child lf_hip_debug_link, origin xyz=0.175 0.105 0 rpy=0 0 0
- added joint lf_hip_joint: type revolute, parent base_link, child lf_hip_link, origin xyz=0.175 0.105 0 rpy=0 0 0, axis 1 0 0, limit lower=-3.14159265359 upper=3.14159265359 effort=25 velocity=1.5
- added joint lh_debug_joint: type fixed, parent base_link, child lh_hip_debug_link, origin xyz=-0.175 0.105 0 rpy=0 0 0
- added joint lh_hip_joint: type revolute, parent base_link, child lh_hip_link, origin xyz=-0.175 0.105 0 rpy=0 0 0, axis 1 0 0, limit lower=-3.14159265359 upper=3.14159265359 effort=25 velocity=1.5
- added joint rf_debug_joint: type fixed, parent base_link, child rf_hip_debug_link, origin xyz=0.175 -0.105 0 rpy=0 0 0
- added joint rf_hip_joint: type revolute, parent base_link, child rf_hip_link, origin xyz=0.175 -0.105 0 rpy=0 0 0, axis 1 0 0, limit lower=-3.14159265359 upper=3.14159265359 effort=25 velocity=1.5
- added joint rh_debug_joint: type fixed, parent base_link, child rh_hip_debug_link, origin xyz=-0.175 -0.105 0 rpy=0 0 0
- added joint rh_hip_joint: type revolute, parent base_link, child rh_hip_link, origin xyz=-0.175 -0.105 0 rpy=0 0 0, axis 1 0 0, limit lower=-3.14159265359 upper=3.14159265359 effort=25 velocity=1.5
- joint lf_lower_leg_joint: axis 0 0 1 -> 0 1 0; limit lower=-3.14159265359 upper=3.14159265359 effort=25 velocity=0.1 -> lower=-3.14159265359 upper=3.14159265359 effort=25 velocity=1.5; origin xyz=0.0 -0.039282 0.0 rpy=0 0 0 -> xyz=0 0 -0.141 rpy=0 0 0
- joint lf_upper_leg_joint: axis 0 0 1 -> 0 1 0; limit lower=-3.14159265359 upper=3.14159265359 effort=25 velocity=0.1 -> lower=-3.14159265359 upper=3.14159265359 effort=25 velocity=1.5; origin xyz=0.083 0.017 -0.092 rpy=0 0 0 -> xyz=0 0.06 0 rpy=0 0 0; parent base_link -> lf_hip_link
- joint lh_lower_leg_joint: axis 0 0 1 -> 0 1 0; limit lower=-3.14159265359 upper=3.14159265359 effort=25 velocity=0.1 -> lower=-3.14159265359 upper=3.14159265359 effort=25 velocity=1.5; origin xyz=0.0 -0.039282 0.0 rpy=0 0 0 -> xyz=0 0 -0.141 rpy=0 0 0
- joint lh_upper_leg_joint: axis 0 0 1 -> 0 1 0; limit lower=-3.14159265359 upper=3.14159265359 effort=25 velocity=0.1 -> lower=-3.14159265359 upper=3.14159265359 effort=25 velocity=1.5; origin xyz=0 0 -0.092 rpy=0 0 0 -> xyz=0 0.06 0 rpy=0 0 0; parent base_link -> lh_hip_link
- joint rf_lower_leg_joint: axis 0 0 1 -> 0 1 0; limit lower=-3.14159265359 upper=3.14159265359 effort=25 velocity=0.1 -> lower=-3.14159265359 upper=3.14159265359 effort=25 velocity=1.5; origin xyz=0.0 -0.039282 0.0 rpy=0 0 0 -> xyz=0 0 -0.141 rpy=0 0 0
- joint rf_upper_leg_joint: axis 0 0 1 -> 0 1 0; limit lower=-3.14159265359 upper=3.14159265359 effort=25 velocity=0.1 -> lower=-3.14159265359 upper=3.14159265359 effort=25 velocity=1.5; origin xyz=.083 .017 0 rpy=0 0 0 -> xyz=0 -0.06 0 rpy=0 0 0; parent base_link -> rf_hip_link
- joint rh_lower_leg_joint: axis 0 0 1 -> 0 1 0; limit lower=-3.14159265359 upper=3.14159265359 effort=25 velocity=0.1 -> lower=-3.14159265359 upper=3.14159265359 effort=25 velocity=1.5; origin xyz=0.0 -0.039282 0.0 rpy=0 0 0 -> xyz=0 0 -0.141 rpy=0 0 0
- joint rh_upper_leg_joint: axis 0 0 1 -> 0 1 0; limit lower=-3.14159265359 upper=3.14159265359 effort=25 velocity=0.1 -> lower=-3.14159265359 upper=3.14159265359 effort=25 velocity=1.5; origin xyz=0 0 0 rpy=0 0 0 -> xyz=0 -0.06 0 rpy=0 0 0; parent base_link -> rh_hip_link
